File: hardware/motor-driver.kicad_sch (KiCad schematic)
At the start: 28 parts, among them J4 Conn_01x06, J5 Conn_01x06, U4 DRV8874PWPR, U5 DRV8874PWPR

Commit message: Moved hardware to separate directory
Other:
- company: (none) -> Sampreet SARKAR
Changed lines of the file:
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@@
 (kicad_sch (version 20211123) (generator eeschema)
   (paper "A4")
+  (title_block
+    (rev "A")
+    (company "Sampreet SARKAR")
+  )
   (junction (at 49.53 44.45) (diameter 0) (color 0 0 0 0)
   )

Commit message: Added pin assignments in firmware
Other:
- title: (none) -> Posit: A STM32 based DC motor controller
Changed lines of the file:
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@@
   (paper "A4")
   (title_block
+    (title "Posit: A STM32 based DC motor controller")
     (rev "A")
     (company "Sampreet SARKAR")

Commit message: Added status LED and silkscreen
Connections:
- net GND: now also U4.17 (GND), U5.17 (GND)
Changed lines of the file:
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@@
   (junction (at 148.59 80.01) (diameter 0) (color 0 0 0 0)
   )
+  (junction (at 148.59 85.09) (diameter 0) (color 0 0 0 0)
+  )
   (junction (at 154.94 121.92) (diameter 0) (color 0 0 0 0)
   )
@@
   )
   (junction (at 49.53 146.05) (diameter 0) (color 0 0 0 0)
+  )
+  (junction (at 148.59 161.29) (diameter 0) (color 0 0 0 0)
   )
   (junction (at 182.88 123.19) (diameter 0) (color 0 0 0 0)
@@
     (stroke (width 0) (type default) (color 0 0 0 0))
   )
+  (wire (pts (xy 148.59 85.09) (xy 148.59 87.63))
+    (stroke (width 0) (type default) (color 0 0 0 0))
+  )
   (wire (pts (xy 148.59 68.58) (xy 148.59 69.85))
     (stroke (width 0) (type default) (color 0 0 0 0))
@@
     (stroke (width 0) (type default) (color 0 0 0 0))
   )
+  (wire (pts (xy 148.59 161.29) (xy 148.59 163.83))
+    (stroke (width 0) (type default) (color 0 0 0 0))
+  )
   (wire (pts (xy 176.53 76.2) (xy 176.53 78.74))
     (stroke (width 0) (type default) (color 0 0 0 0))
@@
     (stroke (width 0) (type default) (color 0 0 0 0))
   )
+  (wire (pts (xy 127 161.29) (xy 148.59 161.29))
+    (stroke (width 0) (type default) (color 0 0 0 0))
+  )
   (wire (pts (xy 82.55 64.77) (xy 91.44 64.77))
     (stroke (width 0) (type default) (color 0 0 0 0))
@@
     (stroke (width 0) (type default) (color 0 0 0 0))
   )
+  (wire (pts (xy 127 85.09) (xy 148.59 85.09))
+    (stroke (width 0) (type default) (color 0 0 0 0))
+  )
   (wire (pts (xy 148.59 133.35) (xy 148.59 139.7))
     (stroke (width 0) (type default) (color 0 0 0 0))
@@
     (stroke (width 0) (type default) (color 0 0 0 0))
   )
-  (wire (pts (xy 148.59 158.75) (xy 148.59 163.83))
+  (wire (pts (xy 148.59 158.75) (xy 148.59 161.29))
     (stroke (width 0) (type default) (color 0 0 0 0))
   )
@@
     (stroke (width 0) (type default) (color 0 0 0 0))
   )
-  (wire (pts (xy 148.59 82.55) (xy 148.59 87.63))
+  (wire (pts (xy 148.59 82.55) (xy 148.59 85.09))
     (stroke (width 0) (type default) (color 0 0 0 0))
   )
@@
     (pin "1")
   )
-  (symbol (lib_id "DRV8874PWPR:DRV8874PWPR") (at 109.22 140.97 0) (unit 1)
+  (symbol (lib_name "DRV8874PWPR_1") (lib_id "DRV8874PWPR:DRV8874PWPR") (at 109.22 140.97 0) (unit 1)
     (in_bom yes) (on_board yes) (fields_autoplaced)
     (property "Reference" "U5" (id 0) (at 109.22 113.03 0))
@@
     (pin "15")
     (pin "16")
+    (pin "17")
     (pin "2")
     (pin "3")
@@
     (pin "14")
     (pin "15")
+    (pin "17")
     (pin "16")
     (pin "2")

Commit message: Minor changes, added 100n cap
Parts:
- added C22, C23: 100n, Capacitor_SMD:C_0603_1608Metric, symbol Device:C_Small
Connections:
- net +12V: now also C22.1, C23.1
- net GND: now also C22.2, C23.2
Changed lines of the file:
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@@
   (junction (at 148.59 80.01) (diameter 0) (color 0 0 0 0)
   )
+  (junction (at 154.94 114.3) (diameter 0) (color 0 0 0 0)
+  )
   (junction (at 148.59 85.09) (diameter 0) (color 0 0 0 0)
   )
@@
   )
   (junction (at 154.94 45.72) (diameter 0) (color 0 0 0 0)
+  )
+  (junction (at 154.94 38.1) (diameter 0) (color 0 0 0 0)
   )
   (junction (at 182.88 46.99) (diameter 0) (color 0 0 0 0)
@@
     (stroke (width 0) (type default) (color 0 0 0 0))
   )
+  (wire (pts (xy 163.83 44.45) (xy 163.83 45.72))
+    (stroke (width 0) (type default) (color 0 0 0 0))
+  )
   (wire (pts (xy 82.55 62.23) (xy 91.44 62.23))
     (stroke (width 0) (type default) (color 0 0 0 0))
@@
     (stroke (width 0) (type default) (color 0 0 0 0))
   )
+  (wire (pts (xy 163.83 121.92) (xy 154.94 121.92))
+    (stroke (width 0) (type default) (color 0 0 0 0))
+  )
   (wire (pts (xy 148.59 161.29) (xy 148.59 163.83))
     (stroke (width 0) (type default) (color 0 0 0 0))
@@
     (stroke (width 0) (type default) (color 0 0 0 0))
   )
+  (wire (pts (xy 163.83 45.72) (xy 154.94 45.72))
+    (stroke (width 0) (type default) (color 0 0 0 0))
+  )
+  (wire (pts (xy 163.83 38.1) (xy 154.94 38.1))
+    (stroke (width 0) (type default) (color 0 0 0 0))
+  )
   (wire (pts (xy 128.27 120.65) (xy 128.27 114.3))
     (stroke (width 0) (type default) (color 0 0 0 0))
@@
     (stroke (width 0) (type default) (color 0 0 0 0))
   )
+  (wire (pts (xy 163.83 39.37) (xy 163.83 38.1))
+    (stroke (width 0) (type default) (color 0 0 0 0))
+  )
   (wire (pts (xy 127 135.89) (xy 137.16 135.89))
     (stroke (width 0) (type default) (color 0 0 0 0))
@@
     (stroke (width 0) (type default) (color 0 0 0 0))
   )
+  (wire (pts (xy 163.83 115.57) (xy 163.83 114.3))
+    (stroke (width 0) (type default) (color 0 0 0 0))
+  )
   (wire (pts (xy 128.27 44.45) (xy 128.27 38.1))
     (stroke (width 0) (type default) (color 0 0 0 0))
@@
     (stroke (width 0) (type default) (color 0 0 0 0))
   )
+  (wire (pts (xy 163.83 114.3) (xy 154.94 114.3))
+    (stroke (width 0) (type default) (color 0 0 0 0))
+  )
   (wire (pts (xy 176.53 58.42) (xy 176.53 68.58))
     (stroke (width 0) (type default) (color 0 0 0 0))
@@
   )
   (wire (pts (xy 49.53 134.62) (xy 49.53 138.43))
+    (stroke (width 0) (type default) (color 0 0 0 0))
+  )
+  (wire (pts (xy 163.83 120.65) (xy 163.83 121.92))
     (stroke (width 0) (type default) (color 0 0 0 0))
   )
@@
     (pin "1")
   )
+  (symbol (lib_id "Device:C_Small") (at 163.83 41.91 0) (unit 1)
+    (in_bom yes) (on_board yes) (fields_autoplaced)
+    (property "Reference" "C22" (id 0) (at 166.37 40.6462 0)
+      (effects (font (size 1.27 1.27)) (justify left))
+    )
+    (property "Value" "100n" (id 1) (at 166.37 43.1862 0)
+      (effects (font (size 1.27 1.27)) (justify left))
+    )
+    (property "Footprint" "Capacitor_SMD:C_0603_1608Metric" (id 2) (at 163.83 41.91 0)
+      (effects (font (size 1.27 1.27)) hide)
+    )
+    (property "Datasheet" "~" (id 3) (at 163.83 41.91 0)
+      (effects (font (size 1.27 1.27)) hide)
+    )
+    (pin "1")
+    (pin "2")
+  )
   (symbol (lib_id "power:+12V") (at 133.35 113.03 0) (unit 1)
     (in_bom yes) (on_board yes)
@@
     )
     (property "Datasheet" "~" (id 3) (at 133.35 43.18 0)
+      (effects (font (size 1.27 1.27)) hide)
+    )
+    (pin "1")
+    (pin "2")
+  )
+  (symbol (lib_id "Device:C_Small") (at 163.83 118.11 0) (unit 1)
+    (in_bom yes) (on_board yes) (fields_autoplaced)
+    (property "Reference" "C23" (id 0) (at 166.37 116.8462 0)
+      (effects (font (size 1.27 1.27)) (justify left))
+    )
+    (property "Value" "100n" (id 1) (at 166.37 119.3862 0)
+      (effects (font (size 1.27 1.27)) (justify left))
+    )
+    (property "Footprint" "Capacitor_SMD:C_0603_1608Metric" (id 2) (at 163.83 118.11 0)
+      (effects (font (size 1.27 1.27)) hide)
+    )
+    (property "Datasheet" "~" (id 3) (at 163.83 118.11 0)
       (effects (font (size 1.27 1.27)) hide)
     )
@@
     (pin "14")
     (pin "15")
+    (pin "16")
     (pin "17")
-    (pin "16")
     (pin "2")
     (pin "3")

Commit message: Updated hardware design, added TagConnect Probe and Battery Voltage Measurement
Parts:
- J4, J5: value Conn_01x06 -> JST-EH_B6B; footprint Connector_JST:JST_PH_S6B-PH-K_1x06_P2.00mm_Horizontal -> Connector_JST:JST_EH_B6B-EH-A_1x06_P2.50mm_Vertical

Commit message: Cleaned up debug firmware
Parts:
- R3: value 10k -> 10k/DNP
Connections:
- net GND: now also U4.7 (IMODE)
- no-connect marks 4 -> 3
Changed lines of the file:
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@@
   (junction (at 140.97 38.1) (diameter 0) (color 0 0 0 0)
   )
-  (no_connect (at 91.44 59.69))
   (no_connect (at 91.44 74.93))
   (no_connect (at 91.44 135.89))
@@
     (stroke (width 0) (type default))
   )
+  (wire (pts (xy 72.39 64.77) (xy 72.39 59.69))
+    (stroke (width 0) (type default))
+  )
   (wire (pts (xy 232.41 139.7) (xy 232.41 144.78))
     (stroke (width 0) (type default))
@@
   )
   (wire (pts (xy 163.83 115.57) (xy 163.83 114.3))
+    (stroke (width 0) (type default))
+  )
+  (wire (pts (xy 72.39 59.69) (xy 91.44 59.69))
     (stroke (width 0) (type default))
   )
@@
   (symbol (lib_id "Device:R_Small") (at 49.53 64.77 0) (unit 1)
     (in_bom yes) (on_board yes) (dnp no) (fields_autoplaced)
-    (property "Reference" "R3" (at 52.07 63.4999 0)
-      (effects (font (size 1.27 1.27)) (justify left))
-    )
-    (property "Value" "10k" (at 52.07 66.0399 0)
+    (property "Reference" "R3" (at 52.07 63.5 0)
+      (effects (font (size 1.27 1.27)) (justify left))
+    )
+    (property "Value" "10k/DNP" (at 52.07 66.04 0)
       (effects (font (size 1.27 1.27)) (justify left))
     )
@@
         )
       )
+    )
+  )
+  (symbol (lib_id "power:GND") (at 72.39 64.77 0) (unit 1)
+    (in_bom yes) (on_board yes) (dnp no) (fields_autoplaced)
+    (property "Reference" "#PWR060" (at 72.39 71.12 0)
+      (effects (font (size 1.27 1.27)) hide)
+    )
+    (property "Value" "GND" (at 72.39 69.85 0)
+      (effects (font (size 1.27 1.27)))
+    )
+    (property "Footprint" "" (at 72.39 64.77 0)
+      (effects (font (size 1.27 1.27)) hide)
+    )
+    (property "Datasheet" "" (at 72.39 64.77 0)
+      (effects (font (size 1.27 1.27)) hide)
+    )
+    (pin "1")
+    (instances
+      (project "four-layer-board"
+        (path "/1cb1f541-eb62-44d7-acc9-294b6c5bea68/66d5fe93-feea-4c1f-9c18-d27390976820"
+          (reference "#PWR060") (unit 1)
+        )
+      )
